Commit message: updates

File: dual_arm_moveit_config/config/dual_arm_world.urdf.xacro (robot description, xacro)
@@ -826,5 +826,5 @@
   </joint>
   <joint name="screwdriver_tcp_joint" type="fixed">
-    <origin rpy="0 0 0" xyz="0 0 -0.24"/>
+    <origin rpy="0 0 0" xyz="0 0 -0.178"/>
     <parent link="screwdriver_base_link"/>
     <child link="screwdriver_tcp"/>

Commit message: Align dual-arm MoveIt configs and update teleop stack

File: dual_arm_moveit_config/config/dual_arm_world.urdf.xacro (robot description, xacro)
@@ -1,848 +1,14 @@
-<?xml version="1.0" ?>
-<!-- =================================================================================== -->
-<!-- |    This document was autogenerated by xacro from dual_arm_scene_description/urdf/dual_srm_scene_mimic.xacro | -->
-<!-- |    EDITING THIS FILE BY HAND IS NOT RECOMMENDED                                 | -->
-<!-- =================================================================================== -->
+<?xml version="1.0"?>
 <robot name="dual_arm_world" xmlns:xacro="http://www.ros.org/wiki/xacro">
   <xacro:arg name="hardware_type" default="fake"/>
   <xacro:arg name="joint_commands_topic" default="/isaac_joint_commands"/>
   <xacro:arg name="joint_states_topic" default="/isaac_joint_states"/>
+  <xacro:include filename="$(find dual_arm_scene_description)/urdf/dual_arm_scene_mimic.xacro"/>
   <xacro:include filename="ros2_control.xacro"/>
   <link name="world"/>
   <joint name="world_fixed" type="fixed">
-    <origin rpy="0 0 0" xyz="0 0 0"/>
+    <origin xyz="0 0 0" rpy="0 0 0"/>
     <parent link="world"/>
     <child link="base_link"/>
-  </joint>
-  <link name="base_link">
-    <visual name="base_link_visual">
-      <origin rpy="0 0 0" xyz="0 0 0"/>
-      <geometry>
-        <mesh filename="package://dual_arm_scene_description/meshes/base_link.stl"/>
-      </geometry>
-      <material name="base_link-material">
-        <color rgba="0.6 0.6 0.6 1.0"/>
-      </material>
-    </visual>
-    <collision name="base_link_collision">
-      <origin rpy="0 0 0" xyz="0 0 0"/>
-      <geometry>
-        <mesh filename="package://dual_arm_scene_description/meshes/base_link.stl"/>
-      </geometry>
-    </collision>
-    <inertial>
-      <mass value="549.24217"/>
-      <inertia ixx="733.29925" ixy="10.147329" ixz="-0.50042511" iyy="218.6186" iyz="-1.0615484" izz="856.04667"/>
-      <origin rpy="0 0 0" xyz="1.1342409 -0.022106511 0.66159052"/>
-    </inertial>
-  </link>
-  <link name="uf850_mount">
-    <visual name="uf850_mount_visual">
-      <origin rpy="0 0 0" xyz="0 0 0"/>
-      <geometry>
-        <mesh filename="package://dual_arm_scene_description/meshes/uf850_mount.stl"/>
-      </geometry>
-      <material name="uf850_mount-material">
-        <color rgba="0.6 0.6 0.6 1.0"/>
-      </material>
-    </visual>
-    <collision name="uf850_mount_collision">
-      <origin rpy="0 0 0" xyz="0 0 0"/>
-      <geometry>
-        <mesh filename="package://dual_arm_scene_description/meshes/uf850_mount.stl"/>
-      </geometry>
-    </collision>
-    <inertial>
-      <mass value="0.91397158"/>
-      <inertia ixx="0.0064874" ixy="0" ixz="0" iyy="0.0032770648" iyz="0" izz="0.0097492319"/>
-      <origin rpy="0 0 0" xyz="0.08 -0.115 -0.005"/>
-    </inertial>
-  </link>
-  <link name="uf_linear_slide">
-    <visual name="uf_linear_slide_visual">
-      <origin rpy="0 0 0" xyz="0 0 0"/>
-      <geometry>
-        <mesh filename="package://dual_arm_scene_description/meshes/uf_linear_slide.stl"/>
-      </geometry>
-      <material name="uf_linear_slide-material">
-        <color rgba="0.6 0.6 0.6 1.0"/>
-      </material>
-    </visual>
-    <collision name="uf_linear_slide_collision">
-      <origin rpy="0 0 0" xyz="0 0 0"/>
-      <geometry>
-        <mesh filename="package://dual_arm_scene_description/meshes/uf_linear_slide.stl"/>
-      </geometry>
-    </collision>
-    <inertial>
-      <mass value="13.780609"/>
-      <inertia ixx="1.4800795" ixy="-0.011257312" ixz="0.0017214077" iyy="0.047827573" iyz="0.010344226" izz="1.5098231"/>
-      <origin rpy="0 0 0" xyz="0.11762264 0.41988986 0.057871539"/>
-    </inertial>
-  </link>
-  <link name="uf850_base_link">
-    <visual name="uf850_base_link_visual">
-      <origin rpy="0 0 0" xyz="0 0 0"/>
-      <geometry>
-        <mesh filename="package://dual_arm_scene_description/meshes/uf850_base_link.stl"/>
-      </geometry>
-      <material name="uf850_base_link-material">
-        <color rgba="0.2 0.2 0.2 1.0"/>
-      </material>
-    </visual>
-    <collision name="uf850_base_link_collision">
-      <origin rpy="0 0 0" xyz="0 0 0"/>
-      <geometry>
-        <mesh filename="package://dual_arm_scene_description/meshes/uf850_base_link.stl"/>
-      </geometry>
-    </collision>
-    <inertial>
-      <mass value="6.1347631"/>
-      <inertia ixx="0.025885384" ixy="-8.6579761e-06" ixz="0.00018118802" iyy="0.026065474" iyz="3.5894686e-06" izz="0.013220454"/>
-      <origin rpy="0 0 0" xyz="-0.00053628339 -1.3586888e-05 -0.085936381"/>
-    </inertial>
-  </link>
-  <link name="robot_base">
-    <visual name="robot_base_visual">
-      <origin rpy="0 0 0" xyz="0 0 0"/>
-      <geometry>
-        <mesh filename="package://dual_arm_scene_description/meshes/robot_base.stl"/>
-      </geometry>
-      <material name="robot_base-material">
-        <color rgba="0.6 0.6 0.6 1.0"/>
-      </material>
-    </visual>
-    <collision name="robot_base_collision">
-      <origin rpy="0 0 0" xyz="0 0 0"/>
-      <geometry>
-        <mesh filename="package://dual_arm_scene_description/meshes/robot_base.stl"/>
-      </geometry>
-    </collision>
-    <inertial>
-      <mass value="3.0226509"/>
-      <inertia ixx="0.008081761" ixy="0.00014252542" ixz="-8.059066e-05" iyy="0.013190464" iyz="-0.00016414733" izz="0.0076576256"/>
-      <origin rpy="0 0 0" xyz="0.042237311 0.016079055 -0.080030822"/>
-    </inertial>
-  </link>
-  <link name="uf850_link1">
-    <visual name="uf850_link1_visual">
-      <origin rpy="0 0 0" xyz="0 0 0"/>
-      <geometry>
-        <mesh filename="package://dual_arm_scene_description/meshes/uf850_link1.stl"/>
-      </geometry>
-      <material name="uf850_link1-material">
-        <color rgba="0.2 0.2 0.2 1.0"/>
-      </material>
-    </visual>
-    <collision name="uf850_link1_collision">
-      <origin rpy="0 0 0" xyz="0 0 0"/>
-      <geometry>
-        <mesh filename="package://dual_arm_scene_description/meshes/uf850_link1.stl"/>
-      </geometry>
-    </collision>
-    <inertial>
-      <mass value="6.9729982"/>
-      <inertia ixx="0.043536443" ixy="2.0332184e-07" ixz="-1.851567e-06" iyy="0.039070397" iyz="-0.0087134974" izz="0.016947432"/>
-      <origin rpy="0 0 0" xyz="-1.8025511e-07 -0.034154821 -0.12261622"/>
-    </inertial>
-  </link>
-  <link name="xarm5_base_link">
-    <visual name="xarm5_base_link_visual">
-      <origin rpy="0 0 0" xyz="0 0 0"/>
-      <geometry>
-        <mesh filename="package://dual_arm_scene_description/meshes/xarm5_base_link.stl"/>
-      </geometry>
-      <material name="xarm5_base_link-material">
-        <color rgba="0.2 0.2 0.2 1.0"/>
-      </material>
-    </visual>
-    <collision name="xarm5_base_link_collision">
-      <origin rpy="0 0 0" xyz="0 0 0"/>
-      <geometry>
-        <mesh filename="package://dual_arm_scene_description/meshes/xarm5_base_link.stl"/>
-      </geometry>
-    </collision>
-    <inertial>
-      <mass value="3.1583482"/>
-      <inertia ixx="0.0085658784" ixy="-2.024796e-05" ixz="0.00021895582" iyy="0.0088387465" iyz="1.3252924e-05" izz="0.0040557663"/>
-      <origin rpy="0 0 0" xyz="-0.0014979471 -9.0589713e-05 -0.073474016"/>
-    </inertial>
-  </link>
-  <link name="uf850_link2">
-    <visual name="uf850_link2_visual">
-      <origin rpy="0 0 0" xyz="0 0 0"/>
-      <geometry>
-        <mesh filename="package://dual_arm_scene_description/meshes/uf850_link2.stl"/>
-      </geometry>
-      <material name="uf850_link2-material">
-        <color rgba="0.2 0.2 0.2 1.0"/>
-      </material>
-    </visual>
-    <collision name="uf850_link2_collision">
-      <origin rpy="0 0 0" xyz="0 0 0"/>
-      <geometry>
-        <mesh filename="package://dual_arm_scene_description/meshes/uf850_link2.stl"/>
-      </geometry>
-    </collision>
-    <inertial>
-      <mass value="10.601221"/>
-      <inertia ixx="0.2482622" ixy="-7.1542664e-05" ixz="1.0682502e-05" iyy="0.020311329" iyz="0.011299878" izz="0.24261629"/>
-      <origin rpy="0 0 0" xyz="7.3435267e-05 -0.2030649 -0.016982096"/>
-    </inertial>
-  </link>
-  <link name="xarm5_link1">
-    <visual name="xarm5_link1_visual">
-      <origin rpy="0 0 0" xyz="0 0 0"/>
-      <geometry>
-        <mesh filename="package://dual_arm_scene_description/meshes/xarm5_link1.stl"/>
-      </geometry>
-      <material name="xarm5_link1-material">
-        <color rgba="0.2 0.2 0.2 1.0"/>
-      </material>
-    </visual>
-    <collision name="xarm5_link1_collision">
-      <origin rpy="0 0 0" xyz="0 0 0"/>
-      <geometry>
-        <mesh filename="package://dual_arm_scene_description/meshes/xarm5_link1.stl"/>
-      </geometry>
-    </collision>
-    <inertial>
-      <mass value="3.5791665"/>
-      <inertia ixx="0.010550565" ixy="8.177212e-06" ixz="2.0212036e-05" iyy="0.0087399248" iyz="-0.0011146261" izz="0.0059189553"/>
-      <origin rpy="0 0 0" xyz="0.00021235348 -0.0073942765 -0.085087873"/>
-    </inertial>
-  </link>
-  <link name="uf850_link3">
-    <visual name="uf850_link3_visual">
-      <origin rpy="0 0 0" xyz="0 0 0"/>
-      <geometry>
-        <mesh filename="package://dual_arm_scene_description/meshes/uf850_link3.stl"/>
-      </geometry>
-      <material name="uf850_link3-material">
-        <color rgba="0.2 0.2 0.2 1.0"/>
-      </material>
-    </visual>
-    <collision name="uf850_link3_collision">
-      <origin rpy="0 0 0" xyz="0 0 0"/>
-      <geometry>
-        <mesh filename="package://dual_arm_scene_description/meshes/uf850_link3.stl"/>
-      </geometry>
-    </collision>
-    <inertial>
-      <mass value="5.23551"/>
-      <inertia ixx="0.021597943" ixy="0.013073745" ixz="-0.010248815" iyy="0.031115493" iyz="0.0062938513" izz="0.037495841"/>
-      <origin rpy="0 0 0" xyz="0.086353664 -0.048344011 0.00055238284"/>
-    </inertial>
-  </link>
-  <link name="xarm5_link2">
-    <visual name="xarm5_link2_visual">
-      <origin rpy="0 0 0" xyz="0 0 0"/>
-      <geometry>
-        <mesh filename="package://dual_arm_scene_description/meshes/xarm5_link2.stl"/>
-      </geometry>
-      <material name="xarm5_link2-material">
-        <color rgba="0.2 0.2 0.2 1.0"/>
-      </material>
-    </visual>
-    <collision name="xarm5_link2_collision">
-      <origin rpy="0 0 0" xyz="0 0 0"/>
-      <geometry>
-        <mesh filename="package://dual_arm_scene_description/meshes/xarm5_link2.stl"/>
-      </geometry>
-    </collision>
-    <inertial>
-      <mass value="7.2722633"/>
-      <inertia ixx="0.082610262" ixy="-0.011770775" ixz="-0.0021405121" iyy="0.023710208" iyz="-0.020572966" izz="0.073292367"/>
-      <origin rpy="0 0 0" xyz="0.013521662 0.16507498 0.048718175"/>
-    </inertial>
-  </link>
-  <link name="uf850_link4">
-    <visual name="uf850_link4_visual">
-      <origin rpy="0 0 0" xyz="0 0 0"/>
-      <geometry>
-        <mesh filename="package://dual_arm_scene_description/meshes/uf850_link4.stl"/>
-      </geometry>
-      <material name="uf850_link4-material">
-        <color rgba="0.2 0.2 0.2 1.0"/>
-      </material>
-    </visual>
-    <collision name="uf850_link4_collision">
-      <origin rpy="0 0 0" xyz="0 0 0"/>
-      <geometry>
-        <mesh filename="package://dual_arm_scene_description/meshes/uf850_link4.stl"/>
-      </geometry>
-    </collision>
-    <inertial>
-      <mass value="4.0108671"/>
-      <inertia ixx="0.035970331" ixy="1.6955558e-07" ixz="-4.6731111e-07" iyy="0.030476726" iyz="0.011440433" izz="0.0091258856"/>
-      <origin rpy="0 0 0" xyz="-1.1537079e-06 0.031961306 -0.12982161"/>
-    </inertial>
-  </link>
-  <link name="xarm5_link3">
-    <visual name="xarm5_link3_visual">
-      <origin rpy="0 0 0" xyz="0 0 0"/>
-      <geometry>
-        <mesh filename="package://dual_arm_scene_description/meshes/xarm5_link3.stl"/>
-      </geometry>
-      <material name="xarm5_link3-material">
-        <color rgba="0.2 0.2 0.2 1.0"/>
-      </material>
-    </visual>
-    <collision name="xarm5_link3_collision">
-      <origin rpy="0 0 0" xyz="0 0 0"/>
-      <geometry>
-        <mesh filename="package://dual_arm_scene_description/meshes/xarm5_link3.stl"/>
-      </geometry>
-    </collision>
-    <inertial>
-      <mass value="5.6490394"/>
-      <inertia ixx="0.080376695" ixy="0.0070825826" ixz="-0.0037563174" iyy="0.020081396" iyz="0.024429402" izz="0.070824751"/>
-      <origin rpy="0 0 0" xyz="0.068753242 -0.15300411 0.0563031"/>
-    </inertial>
-  </link>
-  <link name="uf850_link5">
-    <visual name="uf850_link5_visual">
-      <origin rpy="0 0 0" xyz="0 0 0"/>
-      <geometry>
-        <mesh filename="package://dual_arm_scene_description/meshes/uf850_link5.stl"/>
-      </geometry>
-      <material name="uf850_link5-material">
-        <color rgba="0.2 0.2 0.2 1.0"/>
-      </material>
-    </visual>
-    <collision name="uf850_link5_collision">
-      <origin rpy="0 0 0" xyz="0 0 0"/>
-      <geometry>
-        <mesh filename="package://dual_arm_scene_description/meshes/uf850_link5.stl"/>
-      </geometry>
-    </collision>
-    <inertial>
-      <mass value="2.1315343"/>
-      <inertia ixx="0.0039613529" ixy="9.2075896e-09" ixz="3.2462041e-09" iyy="0.0021080459" iyz="-3.9430409e-05" izz="0.0037634343"/>
-      <origin rpy="0 0 0" xyz="-7.1926445e-08 -0.0050560953 -0.046841769"/>
-    </inertial>
-  </link>
-  <link name="xarm5_link4">
-    <visual name="xarm5_link4_visual">
-      <origin rpy="0 0 0" xyz="0 0 0"/>
-      <geometry>
-        <mesh filename="package://dual_arm_scene_description/meshes/xarm5_link4.stl"/>
-      </geometry>
-      <material name="xarm5_link4-material">
-        <color rgba="0.2 0.2 0.2 1.0"/>
-      </material>
-    </visual>
-    <collision name="xarm5_link4_collision">
-      <origin rpy="0 0 0" xyz="0 0 0"/>
-      <geometry>
-        <mesh filename="package://dual_arm_scene_description/meshes/xarm5_link4.stl"/>
-      </geometry>
-    </collision>
-    <inertial>
-      <mass value="1.9522702"/>
-      <inertia ixx="0.002272531" ixy="0.00058789752" ixz="-0.00074644602" iyy="0.003927311" iyz="0.00019643157" izz="0.0045049523"/>
-      <origin rpy="0 0 0" xyz="0.048945115 -0.01137903 -0.013354913"/>
-    </inertial>
-  </link>
-  <link name="uf850_link6">
-    <visual name="uf850_link6_visual">
-      <origin rpy="0 0 0" xyz="0 0 0"/>
-      <geometry>
-        <mesh filename="package://dual_arm_scene_description/meshes/uf850_link6.stl"/>
-      </geometry>
-      <material name="uf850_link6-material">
-        <color rgba="0.2 0.2 0.2 1.0"/>
-      </material>
-    </visual>
-    <collision name="uf850_link6_collision">
-      <origin rpy="0 0 0" xyz="0 0 0"/>
-      <geometry>
-        <mesh filename="package://dual_arm_scene_description/meshes/uf850_link6.stl"/>
-      </geometry>
-    </collision>
-    <inertial>
-      <mass value="0.38311395"/>
-      <inertia ixx="0.00018268682" ixy="7.4864006e-07" ixz="2.2296854e-08" iyy="0.00018916833" iyz="-8.0720786e-08" izz="0.00032456541"/>
-      <origin rpy="0 0 0" xyz="-4.7049978e-05 -0.000639241 -0.013226374"/>
-    </inertial>
-  </link>
-  <link name="xarm5_link5">
-    <visual name="xarm5_link5_visual">
-      <origin rpy="0 0 0" xyz="0 0 0"/>
-      <geometry>
-        <mesh filename="package://dual_arm_scene_description/meshes/xarm5_link5.stl"/>
-      </geometry>
-      <material name="xarm5_link5-material">
-        <color rgba="0.2 0.2 0.2 1.0"/>
-      </material>
-    </visual>
-    <collision name="xarm5_link5_collision">
-      <origin rpy="0 0 0" xyz="0 0 0"/>
-      <geometry>
-        <mesh filename="package://dual_arm_scene_description/meshes/xarm5_link5.stl"/>
-      </geometry>
-    </collision>
-    <inertial>
-      <mass value="0.31347631"/>
-      <inertia ixx="0.00014060656" ixy="2.5537431e-13" ixz="6.0283601e-14" iyy="0.00013209912" iyz="-1.2386858e-06" izz="0.00023390056"/>
-      <origin rpy="0 0 0" xyz="-2.5931612e-09 0.00045209427 -0.013211346"/>
-    </inertial>
-  </link>
-  <link name="rg6_base_link">
-    <visual name="rg6_base_link_visual">
-      <origin rpy="0 0 0" xyz="0 0 0"/>
-      <geometry>
-        <mesh filename="package://dual_arm_scene_description/meshes/rg6_base_link.stl"/>
-      </geometry>
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