Commit message: working system update

File: dual_arm_scene_description/urdf/dual_arm_scene.urdf (robot description, URDF)
Before this commit: robot dual_arm_scene, 31 links, 32 joints
Joints:
- joint uf850_joint1: limit lower=-0.625 upper=0.625 effort=200.0 velocity=1 -> lower=-6.2831853 upper=6.2831853 effort=200.0 velocity=1
- joint xarm5_joint1: limit lower=-0.625 upper=0.625 effort=50 velocity=1 -> lower=-6.2831853 upper=6.2831853 effort=50 velocity=1

File: dual_arm_scene_description/urdf/dual_arm_scene.xacro (robot description, xacro)
@@ -726,5 +726,5 @@
       <child link="${prefix}uf850_link5"/>
       <axis xyz="0 0 -1"/>
-      <limit effort="19.0" velocity="1" lower="-2.1542083" upper="2.1542083"/>
+      <limit effort="19.0" velocity="1" lower="-2.1642083" upper="2.1642083"/>
     </joint>
     <joint name="${prefix}xarm5_joint4" type="revolute">

File: dual_arm_scene_description/urdf/dual_arm_scene_mimic.urdf (robot description, URDF)
Before this commit: robot dual_srm_scene_mimic, 31 links, 30 joints
Joints:
- joint uf850_joint1: limit lower=-0.625 upper=0.625 effort=200.0 velocity=1 -> lower=-6.2831853 upper=6.2831853 effort=200.0 velocity=1
- joint xarm5_joint1: limit lower=-0.625 upper=0.625 effort=50 velocity=1 -> lower=-6.2831853 upper=6.2831853 effort=50 velocity=1

File: dual_arm_scene_description/urdf/dual_arm_scene_mimic.xacro (robot description, xacro)
@@ -671,5 +671,5 @@
     <child link="uf850_link1"/>
     <axis xyz="0 0 -1"/>
-    <limit effort="200.0" velocity="1" lower="-0.625" upper="0.625"/>
+    <limit effort="200.0" velocity="1" lower="-6.2831853" upper="6.2831853"/>
   </joint>
   <joint name="xarm5_scene_joint" type="fixed">
@@ -690,5 +690,5 @@
     <child link="xarm5_link1"/>
     <axis xyz="0 0 -1"/>
-    <limit effort="50" velocity="1" lower="-0.625" upper="0.625"/>
+    <limit effort="50" velocity="1" lower="-6.2831853" upper="6.2831853"/>
   </joint>
   <joint name="uf850_joint3" type="revolute">
@@ -725,5 +725,5 @@
     <child link="uf850_link5"/>
     <axis xyz="0 0 -1"/>
-    <limit effort="19.0" velocity="1" lower="-2.1542083" upper="2.1542083"/>
+    <limit effort="19.0" velocity="1" lower="-2.1642083" upper="2.1642083"/>
   </joint>
   <joint name="xarm5_joint4" type="revolute">
